File: ZapPad.kicad_pcb (KiCad board)
At the start: 2 copper layers, 61.9 x 95.2 mm, 21 parts, among them J1 Conn_01x04_Pin, SW1 RotaryEncoder_Switch, U1 XIAO-RP2040-DIP

Commit message: finished pcb
Parts:
- moved U1 1.02 mm to (154.8, 67.7)
Routing:
- net SDA Pin: track 28.7 -> 26.9 mm
- net +3V3: track 21.5 -> 20.5 mm
- net Pot Button 1: track 42.2 -> 43.2 mm
- net Column 0: track 103.3 -> 104.2 mm
